Commit message: added lemon graph library and design the graph for cross scenario

File: model/car.urdf.xacro (robot description, xacro)
@@ -10,5 +10,5 @@
 	    <origin xyz="0 0 0" rpy="0 0 0"/>
 	    <geometry>
-		<mesh filename="file://$(find robot_controller)/model/car.dae" scale="0.015 0.015 0.015"/>
+		<mesh filename="file://$(find robot_controller)/model/car.dae" scale="0.012 0.012 0.012"/>
 	    </geometry>
 	    <material name="blue">
